File: pcb/pico-pulse-gen.kicad_sch (KiCad schematic)
At the start: 39 parts, among them SW1 P1_BTN, SW10 P8_BTN, SW11 OUT1_BTN, SW12 OUT2_BTN, SW13 OUT3_BTN, SW2 P2_BTN, SW3 P3_BTN, SW4 P4_BTN, SW5 P5_BTN, SW6 P6_BTN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

Commit message: wip: pcb layout
Parts:
- added C1: 330n, Capacitor_THT:C_Disc_D3.8mm_W2.6mm_P2.50mm, symbol Device:C
- added C2: 10n, Capacitor_THT:C_Disc_D3.8mm_W2.6mm_P2.50mm, symbol Device:C
- added D13: D_Schottky, Diode_THT:D_DO-34_SOD68_P7.62mm_Horizontal, symbol Device:D_Schottky
- added D14, D15: 1N4001, Diode_THT:D_DO-34_SOD68_P7.62mm_Horizontal, symbol Device:D
- added H1, H2, H3, H4: MountingHole, MountingHole:MountingHole_2.7mm_M2.5, symbol Mechanical:MountingHole
- added J1: MOTM_PWR, connector_motm:connector_motm, symbol Connector:Conn_01x04_Male
- added J2: PWR_CON, Connector_PinHeader_2.54mm:PinHeader_1x04_P2.54mm_Vertical, symbol Connector:Conn_01x04_Male
- added J3: OUT_CON, Connector_PinHeader_2.54mm:PinHeader_1x04_P2.54mm_Vertical, symbol Connector:Conn_01x04_Male
- added J4: EXT_CLK, Connector_PinHeader_2.54mm:PinHeader_1x01_P2.54mm_Vertical, symbol Connector:Conn_01x01_Male
- added R13, R14, R15, R16, R17: 100, Resistor_THT:R_Axial_DIN0207_L6.3mm_D2.5mm_P7.62mm_Horizontal, symbol Device:R
- added U2: LM78L05_TO92, Package_TO_SOT_THT:TO-92_Inline, symbol Regulator_Linear:LM78L05_TO92
- RV1: footprint Resistor_THT:R_Axial_DIN0207_L6.3mm_D2.5mm_P7.62mm_Horizontal -> Potentiometer_THT:Potentiometer_Bourns_PTV09A-1_Single_Vertical
- U1: footprint RPi_Pico:RPi_Pico_SMD_TH -> MCU_RaspberryPi_and_Boards:RPi_Pico_SMD_TH
Connections:
- net GND: now also C1.2, C2.2, D14.1 (K), D15.2 (A), J1.2 (Pin_2), J1.3 (Pin_3), J2.3 (Pin_3), U2.2 (GND)
- net GPIO16: now also R16.1
- net GPIO17: now also R13.1
- net GPIO19: now also R14.1
- net GPIO21: now also R15.1
- net GPIO23: now reaches U1.34 (GPIO28_ADC2)
- net GPIO23: now also R17.2
- net at U1.39 (VSYS): now also D13.1 (K)
- new net: J3.4 (Pin_4), R16.2
- new net: J4.1 (Pin_1), R17.1
- new net: J3.3 (Pin_3), R15.2
- new net: J3.2 (Pin_2), R14.2
- new net: J3.1 (Pin_1), R13.2
- new net +15V: C1.1, D15.1 (K), J1.1 (Pin_1), J2.2 (Pin_2), U2.3 (VI)
- new net +5V: C2.1, D13.2 (A), J2.1 (Pin_1), U2.1 (VO)
- new net -15V: D14.2 (A), J1.4 (Pin_4), J2.4 (Pin_4)
- no-connect marks 15 -> 14
Other:
- note added: "(Actually GPIO 28)"
- moved on the sheet: D10, D11, D12, D9, R10, R11, R12, R9, SW11, SW12, SW13

Commit message: feat: routed pcb
Connections:
- net at R16.2: now also J3.1 (Pin_1); no longer J3.4 (Pin_4)
- net at R15.2: now also J3.4 (Pin_4); no longer J3.3 (Pin_3)
- net at R14.2: now also J3.3 (Pin_3); no longer J3.2 (Pin_2)
- net at R13.2: now also J3.2 (Pin_2); no longer J3.1 (Pin_1)
Changed lines of the file:
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@@
+    (stroke (width 0) (type default) (color 0 0 0 0))
+  )
+  (wire (pts (xy 223.52 163.83) (xy 152.4 163.83))
     (stroke (width 0) (type default) (color 0 0 0 0))
   )
@@
     (stroke (width 0) (type default) (color 0 0 0 0))
   )
-  (wire (pts (xy 200.66 168.91) (xy 152.4 168.91))
-    (stroke (width 0) (type default) (color 0 0 0 0))
-  )
   (wire (pts (xy 101.6 78.74) (xy 113.03 78.74))
     (stroke (width 0) (type default) (color 0 0 0 0))
@@
     (stroke (width 0) (type default) (color 0 0 0 0))
   )
-  (wire (pts (xy 223.52 135.89) (xy 223.52 171.45))
-    (stroke (width 0) (type default) (color 0 0 0 0))
-  )
   (bus (pts (xy 63.5 123.19) (xy 73.66 123.19))
     (stroke (width 0) (type default) (color 0 0 0 0))
@@
     (stroke (width 0) (type default) (color 0 0 0 0))
   )
-  (wire (pts (xy 200.66 135.89) (xy 200.66 168.91))
+  (wire (pts (xy 200.66 135.89) (xy 200.66 171.45))
     (stroke (width 0) (type default) (color 0 0 0 0))
   )
@@
     (stroke (width 0) (type default) (color 0 0 0 0))
   )
-  (wire (pts (xy 177.8 135.89) (xy 177.8 166.37))
+  (wire (pts (xy 177.8 135.89) (xy 177.8 168.91))
     (stroke (width 0) (type default) (color 0 0 0 0))
   )
@@
     (stroke (width 0) (type default) (color 0 0 0 0))
   )
-  (wire (pts (xy 223.52 171.45) (xy 152.4 171.45))
-    (stroke (width 0) (type default) (color 0 0 0 0))
-  )
   (wire (pts (xy 106.68 148.59) (xy 106.68 151.13))
     (stroke (width 0) (type default) (color 0 0 0 0))
@@
     (stroke (width 0) (type default) (color 0 0 0 0))
   )
-  (wire (pts (xy 177.8 166.37) (xy 152.4 166.37))
-    (stroke (width 0) (type default) (color 0 0 0 0))
-  )
   (bus (pts (xy 135.89 123.19) (xy 139.7 123.19))
     (stroke (width 0) (type default) (color 0 0 0 0))
@@
     (stroke (width 0) (type default) (color 0 0 0 0))
   )
-  (wire (pts (xy 152.4 163.83) (xy 153.67 163.83))
-    (stroke (width 0) (type default) (color 0 0 0 0))
-  )
   (bus (pts (xy 115.57 81.28) (xy 115.57 91.44))
     (stroke (width 0) (type default) (color 0 0 0 0))
   )
+  (wire (pts (xy 223.52 135.89) (xy 223.52 163.83))
+    (stroke (width 0) (type default) (color 0 0 0 0))
+  )
   (wire (pts (xy 266.7 34.29) (xy 266.7 48.26))
     (stroke (width 0) (type default) (color 0 0 0 0))
@@
     (stroke (width 0) (type default) (color 0 0 0 0))
   )
-  (wire (pts (xy 153.67 135.89) (xy 153.67 163.83))
-    (stroke (width 0) (type default) (color 0 0 0 0))
-  )
   (bus (pts (xy 58.42 55.88) (xy 58.42 58.42))
     (stroke (width 0) (type default) (color 0 0 0 0))
@@
     (stroke (width 0) (type default) (color 0 0 0 0))
   )
+  (wire (pts (xy 153.67 166.37) (xy 152.4 166.37))
+    (stroke (width 0) (type default) (color 0 0 0 0))
+  )
   (wire (pts (xy 105.41 22.86) (xy 105.41 24.13))
     (stroke (width 0) (type default) (color 0 0 0 0))
@@
     (stroke (width 0) (type default) (color 0 0 0 0))
   )
+  (wire (pts (xy 152.4 168.91) (xy 177.8 168.91))
+    (stroke (width 0) (type default) (color 0 0 0 0))
+  )
   (wire (pts (xy 101.6 50.8) (xy 132.08 50.8))
     (stroke (width 0) (type default) (color 0 0 0 0))
   )
+  (wire (pts (xy 152.4 171.45) (xy 200.66 171.45))
+    (stroke (width 0) (type default) (color 0 0 0 0))
+  )
   (wire (pts (xy 171.45 29.21) (xy 179.07 29.21))
     (stroke (width 0) (type default) (color 0 0 0 0))
   )
+  (wire (pts (xy 153.67 135.89) (xy 153.67 166.37))
+    (stroke (width 0) (type default) (color 0 0 0 0))
+  )
